File: schematic_controller/nes_controller_v1.0_v7.sch (EAGLE design)
At the start: 38 parts

Commit message: changed bigger led hole
Parts:
- C1, C2, C3, C4, C5, C6, C7, C8: device rcl:C-EUC0805K -> rcl@1:C-EUC0805K
- R1, R10, R11, R12, R13, R14, R15, R16, R17, R2, R3, R4, R5, R6, R7, R8, R9: device rcl:R-EU_R1206 -> rcl:R-EU_MELF0207R
Connections:
- net +3V3: no longer A.22, B.22, DOWN.22, LEFT.22, RIGHT.22, SELECT.22, START.22, UP.22
- net 3§4: no longer SELECT.11
- net 4$5: no longer A.11
- net DOWN: now also JP2.8; no longer JP2.10
- net LEFT: now also JP2.10; no longer JP2.3
- net N$3: no longer START.11
- net N$4: no longer B.11
- net N$5: no longer UP.11
- net N$6: no longer DOWN.11
- net N$7: no longer RIGHT.11
- net N$8: no longer LEFT.11
- net RIGHT: now also JP2.13; no longer JP2.8
- net SELECT: now also JP2.2; no longer JP2.12
- net START: now also JP2.3; no longer JP2.13
- net UP: now also JP2.12; no longer JP2.2
