File: schematic_controller/nes_controller_v2.0.brd (EAGLE design)
At the start: 110.2 x 55.9 mm, 39 parts

Commit message: xhanged board layout and board layout eralge v7
Parts:
- moved U$1 28.6 mm to (15.4, 41.0)
Changed lines of the file:
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@@
 <element name="BATT1" library="Taschenlampe" package="BATTERIEHALTER" value="" x="39.37" y="16.51" rot="MR90"/>
 <element name="DOWN" library="Schalter-sh" package="SMDTAST" value="" x="17.29" y="8.33" rot="R180"/>
-<element name="JP1" library="pinhead" package="1X15" value="" x="99.39" y="35.3464" rot="MR270"/>
-<element name="JP2" library="pinhead" package="1X15" value="" x="77.33" y="35.38" rot="MR270"/>
+<element name="JP1" library="pinhead" library_urn="urn:adsk.eagle:library:325" package="1X15" package3d_urn="urn:adsk.eagle:package:22424/2" value="" x="99.39" y="35.3464" rot="MR270"/>
+<element name="JP2" library="pinhead" library_urn="urn:adsk.eagle:library:325" package="1X15" package3d_urn="urn:adsk.eagle:package:22424/2" value="" x="77.33" y="35.38" rot="MR270"/>
 <element name="LED1" library="led" package="LED3MM" value="" x="106.68" y="51.2" rot="MR0"/>
 <element name="LEFT" library="Schalter-sh" package="SMDTAST" value="" x="8.26" y="17.22"/>
@@
 <attribute name="SPICEPREFIX" value="C" x="4.8768" y="5.6896" size="1.778" layer="27" rot="R270" display="off"/>
 </element>
-<element name="U$1" library="HTL-Logo" package="LOGOTOP_8" value="" x="43.4848" y="35.3568"/>
+<element name="U$1" library="HTL-Logo" package="LOGOTOP_8" value="" x="15.4432" y="41.0464"/>
 </elements>
 <signals>
